File: pcb/0x42.kicad_pcb (KiCad board)
At the start: 2 copper layers, 285 x 95.1 mm, 261 parts, among them J1 USB_C_Receptacle_USB2.0, J2 ISP, K000 1.5U, K001 1U, K002 1U, K003 1U, K004 1U, K005 1U, K006 1U, K007 1U, K008 1U, K009 1U, K010 1U, K011 1U, K012 1U, K013 1.5U, K100 1.5U, K101 1U, K102 1U, K103 1U, K104 1U, K105 1U, K106 1U, K107 1U, K108 1U, K109 1U, K110 1U, K111 1U, K112 1U, K113 1.5U, K200 1.5U, K201 1U, K202 1U, K203 1U, K204 1U, K205 1U, K206 1U, K207 1U, K208 1U, K209 1U, K210 1U, K211 1U, K212 1U, K213 1.5U, K300 1.5U, K301 1U, K302 1U, K303 1U, K304 1U, K305 1U, K306 1U, K307 1U, K308 1U, K309 1U, K310 1U, K311 1U, K312 1U, K313 1.5U, K400 1.5U, K401 1U, K402 1U, K403 1U, K404 1U, K405 1U, K406 1U, K407 1U, K408 1U, K409 1U, K410 1U, K411 1U, K412 1U, K413 1.5U, Q1 2N7002, SW1 ~Reset, U1 ATmega32U4-MU, U2 PRTR5V0U2X, Y1 Crystal_GND24

Commit message: Complete STM32 PCB v1
Parts:
- removed the C11 at (50.5, 178.8)
- removed the C9 at (61.0, 191.3)
- removed H1: MountingHole_Pad, MountingHole:MountingHole_2.5mm_Pad
- removed LED0, LED1, LED2, LED3, LED4, LED5, LED6: SK6812MINI, 0xLib_LED_SMD:LED_SK6812MINI_PLCC4_3.5x3.5mm_P1.75mm
- removed Q1: 2N7002, Package_TO_SOT_SMD:SOT-23
- removed R000, R001, R002, R003, R004, R005, R006, R007, R008, R009, R010, R011, R012, R013, R100, R101, R102, R103, R104, R105, R106, R107, R108, R109, R110, R111, R112, R113, R200, R201, R202, R203, R204, R205, R206, R207, R208, R209, R210, R211, R212, R213, R300, R301, R302, R303, R304, R305, R306, R307, R308, R309, R310, R311, R312, R313, R400, R401, R402, R403, R404, R405, R406, R407, R408, R409, R410, R411, R412, R413: 1K, 0xLib_Passive_SMD:R_0603_1608Metric
- removed REF**: 60_Outline_Ortho, 0xLib_MK_Boards:60_Outline_Ortho
- removed Y1: Crystal_GND24, Crystal:Crystal_SMD_SeikoEpson_FA238-4Pin_3.2x2.5mm
- added BRD0: MK_Board, 0xLib_MK_Boards:60_Outline_Ortho, F.Cu at (212.0, 116.0)
- added C0: 4n7, 0xLib_Passive_SMD:C_0805_2012Metric, B.Cu at (81.0, 71.6)
- added C6: 10n, 0xLib_Passive_SMD:C_0603_1608Metric, B.Cu at (98.1, 159.6)
- added C8: 100n, 0xLib_Passive_SMD:C_0603_1608Metric, B.Cu at (94.2, 119.8)
- added Cb1: 4µ7, 0xLib_Passive_SMD:C_0805_2012Metric, B.Cu at (77.8, 102.2)
- added Enc0: Rotary_Encoder_Switch, 0xLib_Encoder:RotaryEncoder_Alps_EC11E-Switch_Vertical, F.Cu at (107.2, 154.2)
- added G***: LOGO, 0xLib_Graphics:oshw, B.Cu at (308.0, 125.8)
- added G***: LOGO, 0xLib_Graphics:qmk-powered-by, B.Cu at (243.6, 125.6)
- added G***: LOGO, 0xLib_Graphics:cc-by-nc-sa.eu.noframe, B.Cu at (282.0, 126.0)
- added G***: LOGO, drawings:0x42_82x18mm, F.Cu at (126.2, 116.6)
- added J3: SWD, 0xLib_STM32:ARM_JTAG_SWD_10, B.Cu at (74.7, 131.9)
- added Kb406: 2U, 0xLib_MK_Switches:MXOnly-2U-ReversedStabilizers, F.Cu at (212.0, 154.1)
- added R0: 1M, 0xLib_Passive_SMD:R_0603_1608Metric, B.Cu at (79.1, 71.4)
- added R7: 10K, 0xLib_Passive_SMD:R_0603_1608Metric, B.Cu at (98.1, 156.4)
- added SW2: Boot, 0xLib_Switch_Button:TACT_SWITCH_5.2x5.2_4Pin, B.Cu at (116.8, 120.4)
- added Stab0: 6U, 0xLib_MK_Switches:MXOnly-6U-ReversedStabilizersOnly, F.Cu at (212.0, 154.1)
- added U2: MCP1700-3302E_SOT89, Package_TO_SOT_SMD:SOT-89-3, B.Cu at (77.6, 108.2)
- added U3: IS31FL3731-QF, Package_DFN_QFN:QFN-28-1EP_4x4mm_P0.4mm_EP2.3x2.3mm, B.Cu at (212.0, 90.3)
- C1: value 22p -> 4µ7; footprint 0xLib_Passive_SMD:C_0603_1608Metric -> 0xLib_Passive_SMD:C_0805_2012Metric
- C11: renamed from C8; value 100n -> 1µ
- C12, C13: value 100n -> 4µ7
- C16: value 4n7 -> 1µ
- C2: value 22p -> 1µ
- C3: value 1µ -> 100n
- C4: value 4.7µ -> 100n; footprint 0xLib_Passive_SMD:C_1206_3216Metric -> 0xLib_Passive_SMD:C_0603_1608Metric
- C5, C7: value 100n -> 10n
- J2: value ISP -> Conn_01x04; footprint 0xLib_AVR:ISP_2x03_P2.54mm_Vertical -> Connector_JST:JST_SH_SM04B-SRSS-TB_1x04-1MP_P1.00mm_Horizontal
- K000: footprint 0xLib_MK_Switches:MXOnly-1.5U-Vertical -> 0xLib_MK_Switches:MXOnly-1.5U-Vertical-Flipped
- R1: value 10k -> 10K
- R10: value 330 -> 22K
- R11: value 1M -> 10K
- R2: value 10k -> 5.1k
- R3: value 22 -> 5.1k
- R4: value 22 -> 10K
- R5, R6: value 5.1k -> 10K
- R8: value 100 -> 4K7
- R9: value 10k -> 4K7
- SW1: value ~Reset -> Reset
- U1: value ATmega32U4-MU -> STM32F072CBUx; footprint Package_DFN_QFN:QFN-44-1EP_7x7mm_P0.5mm_EP5.2x5.2mm -> Package_DFN_QFN:QFN-48-1EP_7x7mm_P0.5mm_EP5.6x5.6mm
- moved D213 254.0 mm to (335.0, 108.0)
- moved D313 235.1 mm to (335.0, 143.8)
- moved D212 232.2 mm to (311.2, 108.0)
- moved D211 215.5 mm to (292.2, 108.0)
- moved D312 211.0 mm to (311.2, 143.8)
- moved D413 205.8 mm to (335.0, 146.2)
- moved D210 199.5 mm to (273.1, 108.0)
- moved C15 195.1 mm to (211.4, 86.0), turned to 225 degrees
- moved R10 192.3 mm to (216.6, 88.2), turned to 180 degrees
- moved D311 187.6 mm to (292.2, 143.8)
- moved C14 185.8 mm to (212.0, 95.1)
- moved D209 183.0 mm to (254.1, 108.0)
- moved D013 183.0 mm to (335.0, 86.6)
- moved C16 182.4 mm to (210.2, 84.8), turned to 225 degrees
- moved R11 177.6 mm to (216.6, 86.5), turned to 180 degrees
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- renumbered C6 to C9, U2 to D1
Connections:
- C1 pad 1: /XTAL1 -> +5V
- C10 pad 1: +5V -> +3V3
- C11 pad 1: +5V -> +3V3
- C12 pad 1: +5V -> +3V3
- C13 pad 1: +5V -> +3V3
- C14 pad 1: +5V -> Net-(C14-Pad1)
- C16 pad 1: Shield -> +5V
- C2 pad 1: /XTAL2 -> +3V3
- C3 pad 1: Net-(C3-Pad1) -> NRST
- C4 pad 1: +5V -> BOOT0
- C5 pad 1: +5V -> EncOut_A
- C7 pad 1: +5V -> +3V3
- C9 pad 1: +5V -> +3V3
- D1 pad 2: /BUS_D- -> D-
- D1 pad 3: /BUS_D+ -> D+
- J1 pad A6: /BUS_D+ -> D+
- J1 pad A7: /BUS_D- -> D-
- J1 pad B6: /BUS_D+ -> D+
- J1 pad B7: /BUS_D- -> D-
- J2 pad 1: Row1 -> +5V
- J2 pad 2: +5V -> D-
- J2 pad 3: Row3 -> D+
- J2 pad 4: Row2 -> GND
- K000 pad 3: Net-(K000-Pad3) -> /Key Matrix/CA1
- K000 pad 4: LED_GND -> /Key Matrix/CA7
- K001 pad 3: Net-(K001-Pad3) -> /Key Matrix/CA1
- K001 pad 4: LED_GND -> /Key Matrix/CA6
- K002 pad 3: Net-(K002-Pad3) -> /Key Matrix/CA1
- K002 pad 4: LED_GND -> /Key Matrix/CA5
- K003 pad 3: Net-(K003-Pad3) -> /Key Matrix/CA1
- K003 pad 4: LED_GND -> /Key Matrix/CA4
- K004 pad 3: Net-(K004-Pad3) -> /Key Matrix/CA1
- K004 pad 4: LED_GND -> /Key Matrix/CA3
- K005 pad 3: Net-(K005-Pad3) -> /Key Matrix/CA1
- K005 pad 4: LED_GND -> /Key Matrix/CA2
- K006 pad 3: Net-(K006-Pad3) -> /Key Matrix/CA2
- K006 pad 4: LED_GND -> /Key Matrix/CA1
- K007 pad 3: Net-(K007-Pad3) -> /Key Matrix/CB2
- K007 pad 4: LED_GND -> /Key Matrix/CB1
- K008 pad 3: Net-(K008-Pad3) -> /Key Matrix/CB1
- K008 pad 4: LED_GND -> /Key Matrix/CB2
- K009 pad 3: Net-(K009-Pad3) -> /Key Matrix/CB1
- K009 pad 4: LED_GND -> /Key Matrix/CB3
- K010 pad 3: Net-(K010-Pad3) -> /Key Matrix/CB1
- K010 pad 4: LED_GND -> /Key Matrix/CB4
- K011 pad 3: Net-(K011-Pad3) -> /Key Matrix/CB1
- K011 pad 4: LED_GND -> /Key Matrix/CB5
- K012 pad 3: Net-(K012-Pad3) -> /Key Matrix/CB1
- K012 pad 4: LED_GND -> /Key Matrix/CB6
- K013 pad 3: Net-(K013-Pad3) -> /Key Matrix/CB1
- K013 pad 4: LED_GND -> /Key Matrix/CB7
- K100 pad 3: Net-(K100-Pad3) -> /Key Matrix/CA2
- K100 pad 4: LED_GND -> /Key Matrix/CA7
- K101 pad 3: Net-(K101-Pad3) -> /Key Matrix/CA2
- K101 pad 4: LED_GND -> /Key Matrix/CA6
- K102 pad 3: Net-(K102-Pad3) -> /Key Matrix/CA2
- K102 pad 4: LED_GND -> /Key Matrix/CA5
- K103 pad 3: Net-(K103-Pad3) -> /Key Matrix/CA2
- K103 pad 4: LED_GND -> /Key Matrix/CA4
- K104 pad 3: Net-(K104-Pad3) -> /Key Matrix/CA2
- K104 pad 4: LED_GND -> /Key Matrix/CA3
- K105 pad 3: Net-(K105-Pad3) -> /Key Matrix/CA3
- K105 pad 4: LED_GND -> /Key Matrix/CA2
- K106 pad 3: Net-(K106-Pad3) -> /Key Matrix/CA3
- K106 pad 4: LED_GND -> /Key Matrix/CA1
- K107 pad 3: Net-(K107-Pad3) -> /Key Matrix/CB3
- K107 pad 4: LED_GND -> /Key Matrix/CB1
- K108 pad 3: Net-(K108-Pad3) -> /Key Matrix/CB3
- K108 pad 4: LED_GND -> /Key Matrix/CB2
- K109 pad 3: Net-(K109-Pad3) -> /Key Matrix/CB2
- K109 pad 4: LED_GND -> /Key Matrix/CB3
- K110 pad 3: Net-(K110-Pad3) -> /Key Matrix/CB2
- K110 pad 4: LED_GND -> /Key Matrix/CB4
- K111 pad 3: Net-(K111-Pad3) -> /Key Matrix/CB2
- K111 pad 4: LED_GND -> /Key Matrix/CB5
- K112 pad 3: Net-(K112-Pad3) -> /Key Matrix/CB2
- K112 pad 4: LED_GND -> /Key Matrix/CB6
- K113 pad 3: Net-(K113-Pad3) -> /Key Matrix/CB2
- K113 pad 4: LED_GND -> /Key Matrix/CB7
- K200 pad 3: Net-(K200-Pad3) -> /Key Matrix/CA3
- K200 pad 4: LED_GND -> /Key Matrix/CA7
- K201 pad 3: Net-(K201-Pad3) -> /Key Matrix/CA3
- K201 pad 4: LED_GND -> /Key Matrix/CA6
- K202 pad 3: Net-(K202-Pad3) -> /Key Matrix/CA3
- K202 pad 4: LED_GND -> /Key Matrix/CA5
- K203 pad 3: Net-(K203-Pad3) -> /Key Matrix/CA3
- K203 pad 4: LED_GND -> /Key Matrix/CA4
- K204 pad 3: Net-(K204-Pad3) -> /Key Matrix/CA4
- K204 pad 4: LED_GND -> /Key Matrix/CA3
- K205 pad 3: Net-(K205-Pad3) -> /Key Matrix/CA4
- K205 pad 4: LED_GND -> /Key Matrix/CA2
- K206 pad 3: Net-(K206-Pad3) -> /Key Matrix/CA4
- K206 pad 4: LED_GND -> /Key Matrix/CA1
- K207 pad 3: Net-(K207-Pad3) -> /Key Matrix/CB4
- K207 pad 4: LED_GND -> /Key Matrix/CB1
- K208 pad 3: Net-(K208-Pad3) -> /Key Matrix/CB4
- K208 pad 4: LED_GND -> /Key Matrix/CB2
- K209 pad 3: Net-(K209-Pad3) -> /Key Matrix/CB4
- K209 pad 4: LED_GND -> /Key Matrix/CB3
- K210 pad 3: Net-(K210-Pad3) -> /Key Matrix/CB3
- K210 pad 4: LED_GND -> /Key Matrix/CB4
- K211 pad 3: Net-(K211-Pad3) -> /Key Matrix/CB3
- K211 pad 4: LED_GND -> /Key Matrix/CB5
- K212 pad 3: Net-(K212-Pad3) -> /Key Matrix/CB3
- K212 pad 4: LED_GND -> /Key Matrix/CB6
- K213 pad 3: Net-(K213-Pad3) -> /Key Matrix/CB3
- K213 pad 4: LED_GND -> /Key Matrix/CB7
- K300 pad 3: Net-(K300-Pad3) -> /Key Matrix/CA4
- K300 pad 4: LED_GND -> /Key Matrix/CA7
- K301 pad 3: Net-(K301-Pad3) -> /Key Matrix/CA4
- K301 pad 4: LED_GND -> /Key Matrix/CA6
- K302 pad 3: Net-(K302-Pad3) -> /Key Matrix/CA4
- K302 pad 4: LED_GND -> /Key Matrix/CA5
- K303 pad 3: Net-(K303-Pad3) -> /Key Matrix/CA5
- K303 pad 4: LED_GND -> /Key Matrix/CA4
- K304 pad 3: Net-(K304-Pad3) -> /Key Matrix/CA5
- K304 pad 4: LED_GND -> /Key Matrix/CA3
- K305 pad 3: Net-(K305-Pad3) -> /Key Matrix/CA5
- K305 pad 4: LED_GND -> /Key Matrix/CA2
- K306 pad 3: Net-(K306-Pad3) -> /Key Matrix/CA5
- K306 pad 4: LED_GND -> /Key Matrix/CA1
- K307 pad 3: Net-(K307-Pad3) -> /Key Matrix/CB5
- K307 pad 4: LED_GND -> /Key Matrix/CB1
- K308 pad 3: Net-(K308-Pad3) -> /Key Matrix/CB5
- K308 pad 4: LED_GND -> /Key Matrix/CB2
- K309 pad 3: Net-(K309-Pad3) -> /Key Matrix/CB5
- K309 pad 4: LED_GND -> /Key Matrix/CB3
- K310 pad 3: Net-(K310-Pad3) -> /Key Matrix/CB5
- K310 pad 4: LED_GND -> /Key Matrix/CB4
- K311 pad 3: Net-(K311-Pad3) -> /Key Matrix/CB4
- K311 pad 4: LED_GND -> /Key Matrix/CB5
- K312 pad 3: Net-(K312-Pad3) -> /Key Matrix/CB4
- K312 pad 4: LED_GND -> /Key Matrix/CB6
- K313 pad 3: Net-(K313-Pad3) -> /Key Matrix/CB4
- K313 pad 4: LED_GND -> /Key Matrix/CB7
- K400 pad 3: Net-(K400-Pad3) -> /Key Matrix/CA5
- K400 pad 4: LED_GND -> /Key Matrix/CA7
- K401 pad 3: Net-(K401-Pad3) -> /Key Matrix/CA5
- K401 pad 4: LED_GND -> /Key Matrix/CA6
- K402 pad 3: Net-(K402-Pad3) -> /Key Matrix/CA6
- K402 pad 4: LED_GND -> /Key Matrix/CA5
- K403 pad 3: Net-(K403-Pad3) -> /Key Matrix/CA6
- K403 pad 4: LED_GND -> /Key Matrix/CA4
- K404 pad 3: Net-(K404-Pad3) -> /Key Matrix/CA6
- K404 pad 4: LED_GND -> /Key Matrix/CA3
- K405 pad 3: Net-(K405-Pad3) -> /Key Matrix/CA6
- K405 pad 4: LED_GND -> /Key Matrix/CA2
- K406 pad 3: Net-(K406-Pad3) -> /Key Matrix/CA6
- K406 pad 4: LED_GND -> /Key Matrix/CA1
- K407 pad 3: Net-(K407-Pad3) -> /Key Matrix/CB6
- K407 pad 4: LED_GND -> /Key Matrix/CB1
- K408 pad 3: Net-(K408-Pad3) -> /Key Matrix/CB6
- K408 pad 4: LED_GND -> /Key Matrix/CB2
- K409 pad 3: Net-(K409-Pad3) -> /Key Matrix/CB6
- K409 pad 4: LED_GND -> /Key Matrix/CB3
- K410 pad 3: Net-(K410-Pad3) -> /Key Matrix/CB6
- K410 pad 4: LED_GND -> /Key Matrix/CB4
- K411 pad 3: Net-(K411-Pad3) -> /Key Matrix/CB6
- K411 pad 4: LED_GND -> /Key Matrix/CB5
- K412 pad 3: Net-(K412-Pad3) -> /Key Matrix/CB5
- K412 pad 4: LED_GND -> /Key Matrix/CB6
- K413 pad 3: Net-(K413-Pad3) -> /Key Matrix/CB5
- K413 pad 4: LED_GND -> /Key Matrix/CB7
- Kb106 pad 3: Net-(K106-Pad3) -> /Key Matrix/CA3
- Kb106 pad 4: LED_GND -> /Key Matrix/CA1
- Kb107 pad 3: Net-(K107-Pad3) -> /Key Matrix/CB3
- Kb107 pad 4: LED_GND -> /Key Matrix/CB1
- Kb306 pad 3: Net-(K306-Pad3) -> /Key Matrix/CA5
- Kb306 pad 4: LED_GND -> /Key Matrix/CA1
- Kb307 pad 3: Net-(K307-Pad3) -> /Key Matrix/CB5
- Kb307 pad 4: LED_GND -> /Key Matrix/CB1
- Kb404 pad 3: Net-(K404-Pad3) -> /Key Matrix/CA6
- Kb404 pad 4: LED_GND -> /Key Matrix/CA3
- Kb405 pad 3: Net-(K405-Pad3) -> /Key Matrix/CA6
- Kb405 pad 4: LED_GND -> /Key Matrix/CA2
- Kb408 pad 3: Net-(K408-Pad3) -> /Key Matrix/CB6
- Kb408 pad 4: LED_GND -> /Key Matrix/CB2
- Kb409 pad 3: Net-(K409-Pad3) -> /Key Matrix/CB6
- Kb409 pad 4: LED_GND -> /Key Matrix/CB3
- R1 pad 1: ~RST -> GND
- R1 pad 2: +5V -> BOOT0
- R10 pad 1: Net-(LED0-Pad3) -> GND
- R10 pad 2: LED -> Net-(R10-Pad2)
- R11 pad 2: Shield -> IS31_~SDB
- R2 pad 2: Net-(R2-Pad2) -> Net-(J1-PadA5)
- R3 pad 1: D- -> GND
- R3 pad 2: /BUS_D- -> Net-(J1-PadB5)
- R4 pad 1: D+ -> Enc_A
- R4 pad 2: /BUS_D+ -> +3V3
- R5 pad 1: GND -> EncOut_A
- R5 pad 2: Net-(J1-PadA5) -> Enc_A
- R6 pad 1: GND -> Enc_B
- R6 pad 2: Net-(J1-PadB5) -> +3V3
- R8 pad 1: Net-(Q1-Pad1) -> SDA
- R8 pad 2: /LED_PWM -> +3V3
- R9 pad 1: GND -> SCL
- R9 pad 2: Net-(Q1-Pad1) -> +3V3
- SW1 pad 2: ~RST -> Net-(SW1-Pad2)
- SW1 pad 3: GND -> Net-(SW1-Pad3)
- SW1 pad 4: Net-(SW1-Pad4) -> NRST
- U1 pad 1: Net-(U1-Pad1) -> +3V3
- U1 pad 10: Row2 -> Net-(U1-Pad10)
- U1 pad 11: Row1 -> Net-(U1-Pad11)
- U1 pad 12: Row0 -> Col0
- U1 pad 13: ~RST -> Col7
- U1 pad 14: +5V -> Col8
- U1 pad 15: GND -> Col9
- U1 pad 16: /XTAL2 -> EncOut_A
- U1 pad 17: /XTAL1 -> EncOut_B
- U1 pad 18: Net-(U1-Pad18) -> Row4
- U1 pad 19: Net-(U1-Pad19) -> Row3
- U1 pad 2: +5V -> Net-(U1-Pad2)
- U1 pad 20: Net-(U1-Pad20) -> Row2
- U1 pad 21: Net-(U1-Pad21) -> Row1
- U1 pad 22: Col6 -> Row0
- U1 pad 24: +5V -> +3V3
- U1 pad 25: Col7 -> Col10
- U1 pad 26: Col8 -> Col11
- U1 pad 27: Col9 -> Col12
- U1 pad 28: Col10 -> Col13
- U1 pad 29: Col11 -> Net-(U1-Pad29)
- U1 pad 3: D- -> Net-(U1-Pad3)
- U1 pad 30: Col12 -> Net-(U1-Pad30)
- U1 pad 31: /LED_PWM -> Net-(U1-Pad31)
- U1 pad 32: LED -> D-
- U1 pad 33: Net-(R2-Pad2) -> D+
- U1 pad 34: +5V -> SWDIO
- U1 pad 36: Col0 -> +3V3
- U1 pad 37: Col1 -> SWDCLK
- U1 pad 38: Col2 -> Col6
- U1 pad 39: Col3 -> Col5
- U1 pad 4: D+ -> Net-(U1-Pad4)
- U1 pad 41: Col5 -> Col3
- U1 pad 42: AREF -> Col2
- U1 pad 43: GND -> Col1
- U1 pad 44: +5V -> BOOT0
- U1 pad 45: GND -> SCL
- U1 pad 5: GND -> IS31_~SDB
- U1 pad 6: Net-(C3-Pad1) -> Net-(U1-Pad6)
- U1 pad 7: +5V -> NRST
- U1 pad 8: Row4 -> GND
- U1 pad 9: Row3 -> +3V3
Routing:
- net Row0: track 0.00 -> 362.7 mm, vias 0 -> 10
- net Col13: track 0.00 -> 332.1 mm, vias 0 -> 2
- net /Key Matrix/CB5: track 0.00 -> 319.9 mm, vias 0 -> 1
- net /Key Matrix/CA5: track 0.00 -> 314.0 mm, vias 0 -> 2
- net /Key Matrix/CA3: track 0.00 -> 313.5 mm, vias 0 -> 3
- net Col12: track 0.00 -> 309.4 mm, vias 0 -> 2
- net /Key Matrix/CA6: track 0.00 -> 301.9 mm, vias 0 -> 1
- net Row4: track 0.00 -> 299.2 mm, vias 0 -> 2
- net /Key Matrix/CB6: track 0.00 -> 298.9 mm, vias 0 -> 1
- net Row3: track 0.00 -> 292.7 mm, vias 0 -> 2
- net Col11: track 0.00 -> 289.6 mm, vias 0 -> 2
- net Row1: track 0.00 -> 279.3 mm, vias 0 -> 2
- net Row2: track 0.00 -> 279.2 mm, vias 0 -> 2
- net /Key Matrix/CA1: track 0.00 -> 278.3 mm, vias 0 -> 6
- net /Key Matrix/CB4: track 0.00 -> 278.2 mm, vias 0 -> 1
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- added copper zone on B.Cu, net +5V
- added copper zone on F.Cu, net +5V
- added copper zone on F.Cu, net GND
Other:
- net class Default: clearance 0.2 -> 0.16
- net class PWR: clearance 0.15 -> 0.16
- rule trace_clearance: 0.2 -> 0.16
- board text added: ""Stout Waffle""
- board text added: "0x42"
- board text added: "60% Ortholinear Keyboard PCB - rev0"
- board text added: "Hold Boot during Reset to start in DFU booloader mode"
- board text added: "http://github.com/plut0nium/0x42"
- board text added: "plut0nium 2020"
