File: pcb/key_matrix.sch (KiCad schematic (older format))
At the start: 148 parts, among them K000 1.5U, K001 1U, K002 1U, K003 1U, K004 1U, K005 1U, K006 1U, K007 1U, K008 1U, K009 1U, K010 1U, K011 1U, K012 1U, K013 1.5U, K100 1.5U, K101 1U, K102 1U, K103 1U, K104 1U, K105 1U, K106 1U, K107 1U, K108 1U, K109 1U, K110 1U, K111 1U, K112 1U, K113 1.5U, K200 1.5U, K201 1U, K202 1U, K203 1U, K204 1U, K205 1U, K206 1U, K207 1U, K208 1U, K209 1U, K210 1U, K211 1U, K212 1U, K213 1.5U, K300 1.5U, K301 1U, K302 1U, K303 1U, K304 1U, K305 1U, K306 1U, K307 1U, K308 1U, K309 1U, K310 1U, K311 1U, K312 1U, K313 1.5U, K400 1.5U, K401 1U, K402 1U, K403 1U, K404 1U, K405 1U, K406 1U, K407 1U, K408 1U, K409 1U, K410 1U, K411 1U, K412 1U, K413 1.5U

Commit message: Complete STM32 PCB v1
Parts:
- added C14, C15: 100n, 0xLib_Passive_SMD:C_0603_1608Metric, symbol Device:C
- added C16: 1µ, 0xLib_Passive_SMD:C_0603_1608Metric, symbol Device:C
- added Enc0: Rotary_Encoder_Switch, 0xLib_Encoder:RotaryEncoder_Alps_EC11E-Switch_Vertical, symbol Device:Rotary_Encoder_Switch
- added unit 2 of K000
- added unit 2 of K001
- added unit 2 of K002
- added unit 2 of K003
- added unit 2 of K004
- added unit 2 of K005
- added unit 2 of K006
- added unit 2 of K007
- added unit 2 of K008
- added unit 2 of K009
- added unit 2 of K010
- added unit 2 of K011
- added unit 2 of K012
- added unit 2 of K013
- added unit 2 of K100
- added unit 2 of K101
- added unit 2 of K102
- added unit 2 of K103
- added unit 2 of K104
- added unit 2 of K105
- added unit 2 of K106
- added unit 2 of K107
- added unit 2 of K108
- added unit 2 of K109
- added unit 2 of K110
- added unit 2 of K111
- added unit 2 of K112
- added unit 2 of K113
- added unit 2 of K200
- added unit 2 of K201
- added unit 2 of K202
- added unit 2 of K203
- added unit 2 of K204
- added unit 2 of K205
- added unit 2 of K206
- added unit 2 of K207
- added unit 2 of K208
- added unit 2 of K209
- added unit 2 of K210
- added unit 2 of K211
- added unit 2 of K212
- added unit 2 of K213
- added unit 2 of K300
- added unit 2 of K301
- added unit 2 of K302
- added unit 2 of K303
- added unit 2 of K304
- added unit 2 of K305
- added unit 2 of K306
- added unit 2 of K307
- added unit 2 of K308
- added unit 2 of K309
- added unit 2 of K310
- added unit 2 of K311
- added unit 2 of K312
- added unit 2 of K313
- added unit 2 of K400
- added unit 2 of K401
- added unit 2 of K402
- added unit 2 of K403
- added unit 2 of K404
- added unit 2 of K405
- added unit 2 of K406
- added unit 2 of K407
- added unit 2 of K408
- added unit 2 of K409
- added unit 2 of K410
- added unit 2 of K411
- added unit 2 of K412
- added unit 2 of K413
- added unit 2 of Kb106
- added unit 2 of Kb107
- added unit 2 of Kb306
- added unit 2 of Kb307
- added unit 2 of Kb404
- added unit 2 of Kb405
- added Kb406: 2U, 0xLib_MK_Switches:MXOnly-2U-ReversedStabilizers, symbol 0xLib_MK:Key_Switch_LED
- added unit 2 of Kb408
- added unit 2 of Kb409
- added R10: 22K, 0xLib_Passive_SMD:R_0603_1608Metric, symbol Device:R
- added R11: 10K, 0xLib_Passive_SMD:R_0603_1608Metric, symbol Device:R
- added R8, R9: 4K7, 0xLib_Passive_SMD:R_0603_1608Metric, symbol Device:R
- added Stab0: 6U, 0xLib_MK_Switches:MXOnly-6U-ReversedStabilizersOnly, symbol 0xLib_MK:Stabilizer
- added U3: IS31FL3731-QF, Package_DFN_QFN:QFN-28-1EP_4x4mm_P0.4mm_EP2.3x2.3mm, symbol Driver_LED:IS31FL3731-QF
- K000: footprint 0xLib_MK_Switches:MXOnly-1.5U-Vertical -> 0xLib_MK_Switches:MXOnly-1.5U-Vertical-Flipped
Connections:
- net Col1: now also Enc0.S1
- net Col6: now also Kb406.2
- net at D401.2 (A), K401.1: now also Enc0.S2
- net at D406.2 (A), K406.1: now also Kb406.1
- new net: C14.1, U3.16 (C_FILT)
- new net: R10.2, U3.6 (R_EXT)
- new net +3V3: R8.2, R9.2
- new net +5V: C15.1, C16.1, U3.2 (VCC)
- new net CA1: K000.3 (A), K001.3 (A), K002.3 (A), K003.3 (A), K004.3 (A), K005.3 (A), K006.4 (K), K106.4 (K), K206.4 (K), K306.4 (K), K406.4 (K), Kb106.4 (K), Kb306.4 (K), Kb406.4 (K), U3.21 (CA1)
- new net CA2: K005.4 (K), K006.3 (A), K100.3 (A), K101.3 (A), K102.3 (A), K103.3 (A), K104.3 (A), K105.4 (K), K205.4 (K), K305.4 (K), K405.4 (K), Kb405.4 (K), U3.22 (CA2)
- new net CA3: K004.4 (K), K104.4 (K), K105.3 (A), K106.3 (A), K200.3 (A), K201.3 (A), K202.3 (A), K203.3 (A), K204.4 (K), K304.4 (K), K404.4 (K), Kb106.3 (A), Kb404.4 (K), U3.23 (CA3)
- new net CA4: K003.4 (K), K103.4 (K), K203.4 (K), K204.3 (A), K205.3 (A), K206.3 (A), K300.3 (A), K301.3 (A), K302.3 (A), K303.4 (K), K403.4 (K), U3.24 (CA4)
- new net CA5: K002.4 (K), K102.4 (K), K202.4 (K), K302.4 (K), K303.3 (A), K304.3 (A), K305.3 (A), K306.3 (A), K400.3 (A), K401.3 (A), K402.4 (K), Kb306.3 (A), U3.25 (CA5)
- new net CA6: K001.4 (K), K101.4 (K), K201.4 (K), K301.4 (K), K401.4 (K), K402.3 (A), K403.3 (A), K404.3 (A), K405.3 (A), K406.3 (A), Kb404.3 (A), Kb405.3 (A), Kb406.3 (A), U3.26 (CA6)
- new net CA7: K000.4 (K), K100.4 (K), K200.4 (K), K300.4 (K), K400.4 (K), U3.27 (CA7)
- new net CB1: K007.4 (K), K008.3 (A), K009.3 (A), K010.3 (A), K011.3 (A), K012.3 (A), K013.3 (A), K107.4 (K), K207.4 (K), K307.4 (K), K407.4 (K), Kb107.4 (K), Kb307.4 (K), U3.7 (CB1)
- new net CB2: K007.3 (A), K008.4 (K), K108.4 (K), K109.3 (A), K110.3 (A), K111.3 (A), K112.3 (A), K113.3 (A), K208.4 (K), K308.4 (K), K408.4 (K), Kb408.4 (K), U3.8 (CB2)
- new net CB3: K009.4 (K), K107.3 (A), K108.3 (A), K109.4 (K), K209.4 (K), K210.3 (A), K211.3 (A), K212.3 (A), K213.3 (A), K309.4 (K), K409.4 (K), Kb107.3 (A), Kb409.4 (K), U3.9 (CB3)
- new net CB4: K010.4 (K), K110.4 (K), K207.3 (A), K208.3 (A), K209.3 (A), K210.4 (K), K310.4 (K), K311.3 (A), K312.3 (A), K313.3 (A), K410.4 (K), U3.10 (CB4)
- new net CB5: K011.4 (K), K111.4 (K), K211.4 (K), K307.3 (A), K308.3 (A), K309.3 (A), K310.3 (A), K311.4 (K), K411.4 (K), K412.3 (A), K413.3 (A), Kb307.3 (A), U3.11 (CB5)
- new net CB6: K012.4 (K), K112.4 (K), K212.4 (K), K312.4 (K), K407.3 (A), K408.3 (A), K409.3 (A), K410.3 (A), K411.3 (A), K412.4 (K), Kb408.3 (A), Kb409.3 (A), U3.12 (CB6)
- new net CB7: K013.4 (K), K113.4 (K), K213.4 (K), K313.4 (K), K413.4 (K), U3.13 (CB7)
- new net Enc_A: Enc0.A
- new net Enc_B: Enc0.B
- new net GND: C14.2, C15.2, C16.2, Enc0.C, R10.1, R11.1, U3.18 (AD), U3.29 (GND), U3.5 (GND)
- new net IS31_~SDB: R11.2, U3.3 (~SDB)
- new net SCL: R9.1, U3.20 (SCL)
- new net SDA: R8.1, U3.19 (SDA)
- no-connect marks 0 -> 6
Other:
- note added: "3.3V logic\nwith STM32"
- note added: "6u spacebar stabilizer only\n(switch already covered by other footprints)"
- note added: "LED Driver"
- note added: "LED Matrix"
- note added: "Rotary Encoder"
- note added: "Switch Matrix"
- note added: "~INTB~ not used"
- moved on the sheet: D000, D001, D002, D003, D004, D005, D006, D007, D008, D009, D010, D011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

Commit message: Update Switches and Diodes references on silkscreen
Parts:
- D000, D001, D002, D003, D004, D005, D006, D007, D008, D009, D010, D011, D012, D013, D100, D101, D102, D103, D104, D105, D106, D107, D108, D109, D110, D111, D112, D113, D200, D201, D202, D203, D204, D205, D206, D207, D208, D209, D210, D211, D212, D213, D300, D301, D302, D303, D304, D305, D306, D307, D308, D309, D310, D311, D312, D313, D400, D401, D402, D403, D404, D405, D406, D407, D408, D409, D410, D411, D412, D413: FancyRef (none) -> %true%; LCSC C81598 -> (none)
- K000, K001, K002, K003, K004, K005, K006, K007, K008, K009, K010, K011, K012, K013, K100, K101, K102, K103, K104, K105, K106, K107, K108, K109, K110, K111, K112, K113, K200, K201, K202, K203, K204, K205, K206, K207, K208, K209, K210, K211, K212, K213, K300, K301, K302, K303, K304, K305, K306, K307, K308, K309, K310, K311, K312, K313, K400, K401, K402, K403, K404, K405, K406, K407, K408, K409, K410, K411, K412, K413, Kb106, Kb107, Kb306, Kb307, Kb404, Kb405, Kb406, Kb408, Kb409: FancyRef (none) -> %true%
