File: pcb/key_matrix.sch (KiCad schematic (older format))
At the start: 159 parts, among them K000 1.5U, K001 1U, K002 1U, K003 1U, K004 1U, K005 1U, K006 1U, K007 1U, K008 1U, K009 1U, K010 1U, K011 1U, K012 1U, K013 1.5U, K100 1.5U, K101 1U, K102 1U, K103 1U, K104 1U, K105 1U, K106 1U, K107 1U, K108 1U, K109 1U, K110 1U, K111 1U, K112 1U, K113 1.5U, K200 1.5U, K201 1U, K202 1U, K203 1U, K204 1U, K205 1U, K206 1U, K207 1U, K208 1U, K209 1U, K210 1U, K211 1U, K212 1U, K213 1.5U, K300 1.5U, K301 1U, K302 1U, K303 1U, K304 1U, K305 1U, K306 1U, K307 1U, K308 1U, K309 1U, K310 1U, K311 1U, K312 1U, K313 1.5U, K400 1.5U, K401 1U, K402 1U, K403 1U, K404 1U, K405 1U, K406 1U, K407 1U, K408 1U, K409 1U, K410 1U, K411 1U, K412 1U, K413 1.5U, U3 IS31FL3731-QF

Commit message: Add RGB output - WiP
Parts:
- R10: value 22K -> 22k
- R11: value 10K -> 10k
- R8, R9: value 4K7 -> 4.7k
Changed lines of the file:
@@
 AR Path="/5F3CAEC1/644307F1" Ref="R10"  Part="1"
 F 0 "R10" V 3200 8250 50  0000 C CNN
-F 1 "22K" V 3300 8250 50  0000 C CNN
+F 1 "22k" V 3300 8250 50  0000 C CNN
 F 2 "0xLib_Passive_SMD:R_0603_1608Metric" V 3230 8250 50  0001 C CNN
 F 3 "~" H 3300 8250 50  0001 C CNN
@@
 AR Path="/5F3CAEC1/64430833" Ref="R9"  Part="1"
 F 0 "R9" V 3000 6800 50  0000 C CNN
-F 1 "4K7" V 3100 6800 50  0000 C CNN
+F 1 "4.7k" V 3100 6800 50  0000 C CNN
 F 2 "0xLib_Passive_SMD:R_0603_1608Metric" V 3030 6800 50  0001 C CNN
 F 3 "~" H 3100 6800 50  0001 C CNN
@@
 AR Path="/5F3CAEC1/6443083F" Ref="R8"  Part="1"
 F 0 "R8" V 2800 6800 50  0000 C CNN
-F 1 "4K7" V 2900 6800 50  0000 C CNN
+F 1 "4.7k" V 2900 6800 50  0000 C CNN
 F 2 "0xLib_Passive_SMD:R_0603_1608Metric" V 2830 6800 50  0001 C CNN
 F 3 "~" H 2900 6800 50  0001 C CNN
@@
 AR Path="/5F3CAEC1/64430B91" Ref="R11"  Part="1"
 F 0 "R11" V 2650 8050 50  0000 C CNN
-F 1 "10K" V 2750 8050 50  0000 C CNN
+F 1 "10k" V 2750 8050 50  0000 C CNN
 F 2 "0xLib_Passive_SMD:R_0603_1608Metric" V 2680 8050 50  0001 C CNN
 F 3 "~" H 2750 8050 50  0001 C CNN
