File: pcb/0x42.sch (KiCad schematic (older format))
At the start: 32 parts, among them J1 USB_C_Receptacle_USB2.0, J2 Conn_01x04, J3 SWD_CN4, SW1 Reset, SW2 Boot, U1 STM32F072CBUx, U2 MCP1700-3302E_SOT89

Commit message: Add RGB output - WiP
Parts:
- added J4: Conn_01x03, 0xLib_LED_SMD:RGB_header_VoG_pads, symbol Connector_Generic:Conn_01x03
- added R12: 4.7k, 0xLib_Passive_SMD:R_0603_1608Metric, symbol Device:R
- C0: value 4n7 -> 4.7n
- C1, C12, C13, Cb1: value 4µ7 -> 4.7µ
- R1, R4, R5, R6, R7: value 10K -> 10k
Connections:
- net +5V: now also J4.1 (Pin_1), R12.2
- net Col11: now also U1.29 (PA8); no longer U1.26 (PB13)
- net Col12: now also U1.30 (PA9); no longer U1.27 (PB14)
- net Col13: now also U1.31 (PA10); no longer U1.28 (PB15)
- net GND: now also J4.3 (Pin_3)
- new net RGB_DOUT: J4.2 (Pin_2), R12.1, U1.28 (PB15)
- no-connect marks 12 -> 11
Other:
- note added: "PB15 must be configured\nas open drain output\nfor 5V RGB drive"
- note added: "RGB Interface"
Changed lines of the file:
@@
 P 1200 6750
 F 0 "C0" H 1315 6796 50  0000 L CNN
-F 1 "4n7" H 1315 6705 50  0000 L CNN
+F 1 "4.7n" H 1315 6705 50  0000 L CNN
 F 2 "0xLib_Passive_SMD:C_0805_2012Metric" H 1238 6600 50  0001 C CNN
 F 3 "~" H 1200 6750 50  0001 C CNN
@@
 P 1150 4850
 F 0 "C1" H 1265 4896 50  0000 L CNN
-F 1 "4µ7" H 1265 4805 50  0000 L CNN
+F 1 "4.7µ" H 1265 4805 50  0000 L CNN
 F 2 "0xLib_Passive_SMD:C_0805_2012Metric" H 1188 4700 50  0001 C CNN
 F 3 "~" H 1150 4850 50  0001 C CNN
@@
 P 3950 7000
 F 0 "R1" V 4050 7000 50  0000 C CNN
-F 1 "10K" V 3950 7000 50  0000 C CNN
+F 1 "10k" V 3950 7000 50  0000 C CNN
 F 2 "0xLib_Passive_SMD:R_0603_1608Metric" V 3880 7000 50  0001 C CNN
 F 3 "~" H 3950 7000 50  0001 C CNN
@@
 P 8100 3650
 F 0 "C12" H 8215 3696 50  0000 L CNN
-F 1 "4µ7" H 8215 3605 50  0000 L CNN
+F 1 "4.7µ" H 8215 3605 50  0000 L CNN
 F 2 "0xLib_Passive_SMD:C_0603_1608Metric" H 8138 3500 50  0001 C CNN
 F 3 "~" H 8100 3650 50  0001 C CNN
@@
 P 7300 4700
 F 0 "C13" H 7415 4746 50  0000 L CNN
-F 1 "4µ7" H 7415 4655 50  0000 L CNN
+F 1 "4.7µ" H 7415 4655 50  0000 L CNN
 F 2 "0xLib_Passive_SMD:C_0603_1608Metric" H 7338 4550 50  0001 C CNN
 F 3 "~" H 7300 4700 50  0001 C CNN
@@
 P 7500 1750
 F 0 "R5" V 7400 1750 50  0000 C CNN
-F 1 "10K" V 7500 1750 50  0000 C CNN
+F 1 "10k" V 7500 1750 50  0000 C CNN
 F 2 "0xLib_Passive_SMD:R_0603_1608Metric" V 7430 1750 50  0001 C CNN
 F 3 "~" H 7500 1750 50  0001 C CNN
@@
 P 7700 1750
 F 0 "R7" V 7600 1750 50  0000 C CNN
-F 1 "10K" V 7700 1750 50  0000 C CNN
+F 1 "10k" V 7700 1750 50  0000 C CNN
 F 2 "0xLib_Passive_SMD:R_0603_1608Metric" V 7630 1750 50  0001 C CNN
 F 3 "~" H 7700 1750 50  0001 C CNN
@@
 P 7700 1350
 F 0 "R6" V 7600 1350 50  0000 C CNN
-F 1 "10K" V 7700 1350 50  0000 C CNN
+F 1 "10k" V 7700 1350 50  0000 C CNN
 F 2 "0xLib_Passive_SMD:R_0603_1608Metric" V 7630 1350 50  0001 C CNN
 F 3 "~" H 7700 1350 50  0001 C CNN
@@
 P 7500 1350
 F 0 "R4" V 7400 1350 50  0000 C CNN
-F 1 "10K" V 7500 1350 50  0000 C CNN
+F 1 "10k" V 7500 1350 50  0000 C CNN
 F 2 "0xLib_Passive_SMD:R_0603_1608Metric" V 7430 1350 50  0001 C CNN
 F 3 "~" H 7500 1350 50  0001 C CNN
@@
 P 1450 4850
 F 0 "Cb1" H 1565 4896 50  0000 L CNN
-F 1 "4µ7" H 1565 4805 50  0000 L CNN
+F 1 "4.7µ" H 1565 4805 50  0000 L CNN
 F 2 "0xLib_Passive_SMD:C_0805_2012Metric" H 1488 4700 50  0001 C CNN
 F 3 "~" H 1450 4850 50  0001 C CNN
@@
 Text GLabel 5900 4300 2    50   Input ~ 0
 Col6
-Text GLabel 4200 4300 0    50   Input ~ 0
+Text GLabel 5900 3800 2    50   Input ~ 0
 Col13
 Wire Wire Line
 	5900 4300 5700 4300
-Text GLabel 4200 4200 0    50   Input ~ 0
+Text GLabel 5900 3700 2    50   Input ~ 0
 Col12
-Text GLabel 4200 4100 0    50   Input ~ 0
+Text GLabel 5900 3600 2    50   Input ~ 0
 Col11
-Wire Wire Line
-	4200 4300 4400 4300
-Wire Wire Line
-	4200 4200 4400 4200
-Wire Wire Line
-	4200 4100 4400 4100
 Text GLabel 4200 4000 0    50   Input ~ 0
 Col10
@@
 NoConn ~ 5700 2800
 NoConn ~ 5700 2900
-NoConn ~ 5700 3600
-NoConn ~ 5700 3700
-NoConn ~ 5700 3800
 Wire Wire Line
 	5900 3000 5700 3000
@@
 	5400 6850 5400 6950
 NoConn ~ 5900 6500
+Wire Wire Line
+	5900 3600 5700 3600
+Wire Wire Line
+	5900 3700 5700 3700
+Wire Wire Line
+	5700 3800 5900 3800
+Wire Wire Line
+	4400 4300 4200 4300
+Text GLabel 4200 4300 0    50   Input ~ 0
+RGB_DOUT
+NoConn ~ 4400 4100
+NoConn ~ 4400 4200
+Wire Notes Line
+	8500 5600 8500 6350
+Wire Notes Line
+	8500 6350 6750 6350
+Wire Notes Line
+	6750 6350 6750 5600
+Wire Notes Line
+	6750 5600 8500 5600
+Text Notes 6750 5600 0    70   ~ 0
+RGB Interface
+Text GLabel 7450 6200 0    50   Input ~ 0
+RGB_DOUT
+$Comp
+L power:+5V #PWR0117
+U 1 1 5FDD9A2D
+P 7100 5850
+F 0 "#PWR0117" H 7100 5700 50  0001 C CNN
+F 1 "+5V" H 7115 6023 50  0000 C CNN
+F 2 "" H 7100 5850 50  0001 C CNN
+F 3 "" H 7100 5850 50  0001 C CNN
+	1    7100 5850
+	1    0    0    -1
+$EndComp
+$Comp
+L power:+5V #PWR0121
+U 1 1 5FDDAF97
+P 7800 5850
+F 0 "#PWR0121" H 7800 5700 50  0001 C CNN
+F 1 "+5V" H 7815 6023 50  0000 C CNN
+F 2 "" H 7800 5850 50  0001 C CNN
+F 3 "" H 7800 5850 50  0001 C CNN
+	1    7800 5850
+	1    0    0    -1
+$EndComp
+$Comp
+L Device:R R12
+U 1 1 5FDDBFAF
+P 7350 6000
+F 0 "R12" V 7250 6000 50  0000 C CNN
+F 1 "4.7k" V 7350 6000 50  0000 C CNN
+F 2 "0xLib_Passive_SMD:R_0603_1608Metric" V 7280 6000 50  0001 C CNN
+F 3 "~" H 7350 6000 50  0001 C CNN
+	1    7350 6000
+	0    1    1    0
+$EndComp
+$Comp
+L Connector_Generic:Conn_01x03 J4
+U 1 1 5FDDD7BB
+P 8100 6000
+F 0 "J4" H 8050 6200 50  0000 L CNN
+F 1 "Conn_01x03" V 8200 5750 50  0000 L CNN
+F 2 "0xLib_LED_SMD:RGB_header_VoG_pads" H 8100 6000 50  0001 C CNN
+F 3 "~" H 8100 6000 50  0001 C CNN
+	1    8100 6000
+	1    0    0    -1
+$EndComp
+Wire Wire Line
+	7100 5850 7100 6000
+Wire Wire Line
+	7100 6000 7200 6000
+$Comp
+L power:GND #PWR0122
+U 1 1 5FDEBBC3
+P 7800 6150
+F 0 "#PWR0122" H 7800 5900 50  0001 C CNN
+F 1 "GND" H 7805 5977 50  0000 C CNN
+F 2 "" H 7800 6150 50  0001 C CNN
+F 3 "" H 7800 6150 50  0001 C CNN
+	1    7800 6150
+	1    0    0    -1
+$EndComp
+Wire Wire Line
+	7900 6100 7800 6100
+Wire Wire Line
+	7800 6100 7800 6150
+Wire Wire Line
+	7900 5900 7800 5900
+Wire Wire Line
+	7800 5900 7800 5850
+Wire Wire Line
+	7900 6000 7650 6000
+Wire Wire Line
+	7600 6200 7650 6000
+Wire Wire Line
+	7450 6200 7600 6200
+Connection ~ 7650 6000
+Wire Wire Line
+	7650 6000 7500 6000
+Text Notes 3650 4600 0    40   ~ 0
+PB15 must be configured\nas open drain output\nfor 5V RGB drive
 $EndSCHEMATC
