File: pcb/mechanical.kicad_sch (KiCad schematic)
At the start: 1 part

Commit message: Switched to RP2040 - PCB finalization
Parts:
- BRD0: now left out of the parts list
Changed lines of the file:
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@@
   )
   (symbol (lib_id "0xLib_MK:MK_Board") (at 147.32 63.5 0) (unit 1)
-    (in_bom yes) (on_board yes)
+    (in_bom no) (on_board yes)
     (property "Reference" "BRD0" (id 0) (at 160.7312 63.8048 0)
       (effects (font (size 1.27 1.27)) (justify left))
