File: pcb/0x42.kicad_sch (KiCad schematic)
At the start: 42 parts, among them J1 USB_C_Receptacle_USB2.0, J2 Conn_01x04, J3 Conn_01x03, SW1 Reset, SW2 Boot, U1 RP2040, U2 GD25Q80CEIGR, U3 XC6210B332MR, Y1 Crystal_GND24

Commit message: Update PCB assembly information (mostly part reference numbers)
Parts:
- U2: value GD25Q80CEIGR -> GD25Q80EEIGR; LCSC C395484 -> C2874937
Changed lines of the file:
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@@
       (effects (font (size 1.27 1.27)) (justify left))
     )
-    (property "Value" "GD25Q80CEIGR" (at 247.1294 127 0)
+    (property "Value" "GD25Q80EEIGR" (at 247.1294 127 0)
       (effects (font (size 1.27 1.27)) (justify left))
     )
@@
       (effects (font (size 1.27 1.27)) hide)
     )
-    (property "LCSC" "C395484" (at 245.11 137.16 0)
+    (property "LCSC" "C2874937" (at 245.11 137.16 0)
       (effects (font (size 1.27 1.27)) hide)
     )

Commit message: solved some schematic <> pcb inconsistencies on the encoder interface
Parts:
- removed C15, C16: 10n, 0xLib_Passive_SMD:C_0603_1608Metric, symbol Device:C
- removed R10, R9: 100, 0xLib_Passive_SMD:R_0603_1608Metric, symbol Device:R
- removed R11, R12: 10k, 0xLib_Passive_SMD:R_0603_1608Metric, symbol Device:R
Other:
- sheet Key Matrix ports: added EncOut_A, EncOut_B; removed Enc_A, Enc_B
- note removed: "Encoder interface"
- note removed: "NOTE R11, R12, C15 & C16 not mounted Replace R9 & R10 with 10k if installing filter"
