File: pcb/key_matrix.kicad_sch (KiCad schematic)
At the start: 168 parts, among them K000 1.5U, K001 1U, K002 1U, K003 1U, K004 1U, K005 1U, K006 1U, K007 1U, K008 1U, K009 1U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

Commit message: Alternate LCSC Part # for LL4148
Parts:
- D000, D001, D002, D003, D004, D005, D006, D007, D008, D009, D010, D011, D012, D013, D100, D101, D102, D103, D104, D105, D106, D107, D108, D109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: LCSC C9808 -> C5345986
